File: _electronic/KiCad/e-tkt.kicad_pcb (KiCad board)
At the start: 6 copper layers, 99.6 x 76.2 mm, 122 parts

Commit message: 6v and power latch backup
Parts:
- added C_POW_BST2: 0.33uF 50V, Capacitor_SMD:C_0603_1608Metric_Pad1.08x0.95mm_HandSolder, B.Cu at (168.1, -161.5)
- added C_POW_BST3: 0.1uF 50V, Capacitor_SMD:C_0603_1608Metric_Pad1.08x0.95mm_HandSolder, B.Cu at (177.3, -161.5)
- added JP1: SolderJumper_2_Open, Jumper:SolderJumper-2_P1.3mm_Open_Pad1.0x1.5mm, B.Cu at (149.6, -164.7)
- added JP2: SolderJumper_2_Open, Jumper:SolderJumper-2_P1.3mm_Open_Pad1.0x1.5mm, B.Cu at (149.6, -167.3)
- added J_B_12v_1: TestPoint, TestPoint:TestPoint_Pad_D1.5mm, B.Cu at (170.2, -162.6)
- added J_B_6v_1: TestPoint, TestPoint:TestPoint_Pad_D1.5mm, B.Cu at (175.3, -162.6)
- added J_B_GND_1: TestPoint, TestPoint:TestPoint_Pad_D1.5mm, B.Cu at (172.7, -162.6)
- Q_POW1: value IRLML6302TRPBF -> SQ2351ES-T1_GE3
Routing:
- net +6V: track 149.3 -> 176.5 mm, vias 18 -> 22
- net +12V: track 276.9 -> 282.6 mm
- net GNDREF: vias 361 -> 352
- added copper zone on B.Cu, net Net-(J_POW1-Pad1)
Other:
- board text added: "IN"

Commit message: uln2003 soic narrow
Parts:
- U_STP1: footprint Package_SO:SOIC-16W_5.3x10.2mm_P1.27mm -> Package_SO:SOIC-16_3.9x9.9mm_P1.27mm
Routing:
- net +6V: track 176.5 -> 177.7 mm, vias 22 -> 23
- net Net-(D_STP4-Pad1): track 18.6 -> 19.6 mm
- net Net-(D_STP3-Pad1): track 15.1 -> 16.2 mm
- net Net-(D_STP2-Pad1): track 12.1 -> 13.2 mm
- net Net-(D_STP1-Pad1): track 12.2 -> 13.3 mm
- net IO4 ULN 2: track 44.3 -> 45.4 mm
- net IO2 ULN 3: track 37.6 -> 38.7 mm
- net IO16 ULN 4: track 55.3 -> 56.4 mm
- net IO15 ULN 1: track 33.1 -> 34.2 mm
- net GNDREF: vias 352 -> 347
